Commit message: added ft sensor to the sim

File: mujoco/xarm7/xarm7.urdf (robot description, URDF)
Before this commit: robot xarm7, 8 links, 7 joints
Links:
- added link ft_sensor_link, mass 0.445; visual mesh filename=assets/FTSensor.stl
Joints:
- added joint ft_sensor_joint: type fixed, parent link7, child ft_sensor_link, origin xyz=0 0 0 rpy=0 0 0
